File: LoRaNode.sch (KiCad schematic (older format))
At the start: 60 parts, among them J1 CONN_01X04, J10 D4, J11 A1, J12 A2, J13 A3, J14 D8, J2 Conn_01x06, J3 Conn_01x02, J4 ISP, J5 Conn_01x06, J6 Conn_01x04, J7 USB_B_Micro, J8 D2, J9 D3, U1 RFM95W-868S2, U2 MCP73871, U3 TPS63031, U4 ATMEGA328P-AU, Y1 8MHz HC5032/4

Commit message: Changed Antenna dimension, changed TPS63031 footprint
Parts:
- C1, C2: symbol Arduino_Mini-rescue:C-RESCUE-Arduino_Mini -> LoRaNode-rescue:C-RESCUE-Arduino_Mini-Arduino_Mini-rescue
- J1: symbol Arduino_Mini-rescue:CONN_01X04-RESCUE-Arduino_Mini -> LoRaNode-rescue:CONN_01X04-RESCUE-Arduino_Mini-Arduino_Mini-rescue
- L1: symbol Arduino_Mini-rescue:L-RESCUE-Arduino_Mini -> LoRaNode-rescue:L-RESCUE-Arduino_Mini-Arduino_Mini-rescue
- U1: symbol Arduino_Mini-rescue:RFM95W-868S2-RESCUE-Arduino_Mini -> LoRaNode-rescue:RFM95W-868S2-RESCUE-Arduino_Mini-Arduino_Mini-rescue
- U3: footprint Housings_SON:Texas_S-PVSON-N10 -> Package_SON:Texas_S-PWSON-N10
Other:
- note added: "ToDo:\nChange ground symbols\n"
- note removed: "Change TPS63031 footprint\nShorten last antenna segment\nDuplicate the antenna layout on second layer\nChange ground symbols\n"
Changed lines of the file:
@@
 EESchema Schematic File Version 4
-LIBS:Arduino_Mini-cache
+LIBS:LoRaNode-cache
 EELAYER 26 0
 EELAYER END
@@
 $EndDescr
 $Comp
-L Arduino_Mini-rescue:RFM95W-868S2-RESCUE-Arduino_Mini U1
+L LoRaNode-rescue:RFM95W-868S2-RESCUE-Arduino_Mini-Arduino_Mini-rescue U1
 U 1 1 5A1D2B73
 P 9100 5000
@@
 10(**/SS)
 $Comp
-L Arduino_Mini-rescue:+3.3V-RESCUE-Arduino_Mini #PWR09
+L LoRaNode-rescue:+3.3V-RESCUE-Arduino_Mini-Arduino_Mini-rescue #PWR09
 U 1 1 5A1D2CAF
 P 9100 4450
@@
 ANT
 $Comp
-L Arduino_Mini-rescue:C-RESCUE-Arduino_Mini C1
+L LoRaNode-rescue:C-RESCUE-Arduino_Mini-Arduino_Mini-rescue C1
 U 1 1 5A1D4CFC
 P 9900 4900
@@
 $EndComp
 $Comp
-L Arduino_Mini-rescue:C-RESCUE-Arduino_Mini C2
+L LoRaNode-rescue:C-RESCUE-Arduino_Mini-Arduino_Mini-rescue C2
 U 1 1 5A1D4D32
 P 10350 4900
@@
 $EndComp
 $Comp
-L Arduino_Mini-rescue:L-RESCUE-Arduino_Mini L1
+L LoRaNode-rescue:L-RESCUE-Arduino_Mini-Arduino_Mini-rescue L1
 U 1 1 5A1D4D69
 P 10150 4700
@@
 Connection ~ 10150 5100
 $Comp
-L Arduino_Mini-rescue:CONN_01X04-RESCUE-Arduino_Mini J1
+L LoRaNode-rescue:CONN_01X04-RESCUE-Arduino_Mini-Arduino_Mini-rescue J1
 U 1 1 5A1D6448
 P 7750 5450
@@
 A5
 $Comp
-L Arduino_Mini-rescue:+3.3V-RESCUE-Arduino_Mini #PWR012
+L LoRaNode-rescue:+3.3V-RESCUE-Arduino_Mini-Arduino_Mini-rescue #PWR012
 U 1 1 5A1D670C
 P 7300 5500
@@
 F 0 "U3" H 4250 5000 50  0000 C CNN
 F 1 "TPS63031" H 3850 5000 50  0000 C CNN
-F 2 "Housings_SON:Texas_S-PVSON-N10" H 3850 4600 50  0001 C CNN
+F 2 "Package_SON:Texas_S-PWSON-N10" H 3850 4600 50  0001 C CNN
 F 3 "" H 3850 4600 50  0001 C CNN
 	1    4000 4600
@@
 VOUT
 $Comp
-L Arduino_Mini-rescue:+3.3V-RESCUE-Arduino_Mini #PWR035
+L LoRaNode-rescue:+3.3V-RESCUE-Arduino_Mini-Arduino_Mini-rescue #PWR035
 U 1 1 5B163EAE
 P 5150 4400
@@
 VOUT
 $Comp
-L Arduino_Mini-rescue:+3.3V-RESCUE-Arduino_Mini #PWR036
+L LoRaNode-rescue:+3.3V-RESCUE-Arduino_Mini-Arduino_Mini-rescue #PWR036
 U 1 1 5B16C097
 P 1900 5250
@@
 $EndComp
 $Comp
-L Arduino_Mini-rescue:+3.3V-RESCUE-Arduino_Mini #PWR013
+L LoRaNode-rescue:+3.3V-RESCUE-Arduino_Mini-Arduino_Mini-rescue #PWR013
 U 1 1 5B0B0C8E
 P 7700 1500
@@
 $EndComp
 $Comp
-L Arduino_Mini-rescue:+3.3V-RESCUE-Arduino_Mini #PWR038
+L LoRaNode-rescue:+3.3V-RESCUE-Arduino_Mini-Arduino_Mini-rescue #PWR038
 U 1 1 5B0C4FBD
 P 8500 750
@@
 $EndComp
 $Comp
-L Arduino_Mini-rescue:+3.3V-RESCUE-Arduino_Mini #PWR039
+L LoRaNode-rescue:+3.3V-RESCUE-Arduino_Mini-Arduino_Mini-rescue #PWR039
 U 1 1 5B0C5655
 P 8950 750
@@
 $EndComp
 $Comp
-L Arduino_Mini-rescue:+3.3V-RESCUE-Arduino_Mini #PWR045
+L LoRaNode-rescue:+3.3V-RESCUE-Arduino_Mini-Arduino_Mini-rescue #PWR045
 U 1 1 5B13CB93
 P 10850 3200
@@
 $EndComp
 $Comp
-L Arduino_Mini-rescue:+3.3V-RESCUE-Arduino_Mini #PWR048
+L LoRaNode-rescue:+3.3V-RESCUE-Arduino_Mini-Arduino_Mini-rescue #PWR048
 U 1 1 5B1C9B3E
 P 8050 750
@@
 $EndComp
 $Comp
-L Arduino_Mini-rescue:+3.3V-RESCUE-Arduino_Mini #PWR050
+L LoRaNode-rescue:+3.3V-RESCUE-Arduino_Mini-Arduino_Mini-rescue #PWR050
 U 1 1 5B24C6EF
 P 7350 4500
@@
 $EndComp
 $Comp
-L Arduino_Mini-rescue:+3.3V-RESCUE-Arduino_Mini #PWR052
+L LoRaNode-rescue:+3.3V-RESCUE-Arduino_Mini-Arduino_Mini-rescue #PWR052
 U 1 1 5B24C704
 P 7800 4500
@@
 RES
 $Comp
-L Arduino_Mini-rescue:+3.3V-RESCUE-Arduino_Mini #PWR055
+L LoRaNode-rescue:+3.3V-RESCUE-Arduino_Mini-Arduino_Mini-rescue #PWR055
 U 1 1 5B2D22EF
 P 5650 6550
@@
 $EndComp
 $Comp
-L Arduino_Mini-rescue:+3.3V-RESCUE-Arduino_Mini #PWR058
+L LoRaNode-rescue:+3.3V-RESCUE-Arduino_Mini-Arduino_Mini-rescue #PWR058
 U 1 1 5B309256
 P 6650 6700
@@
 SCL
 $Comp
-L Arduino_Mini-rescue:+3.3V-RESCUE-Arduino_Mini #PWR02
+L LoRaNode-rescue:+3.3V-RESCUE-Arduino_Mini-Arduino_Mini-rescue #PWR02
 U 1 1 5B0862C7
 P 1900 5900
@@
 $EndComp
 $Comp
-L Arduino_Mini-rescue:+3.3V-RESCUE-Arduino_Mini #PWR06
+L LoRaNode-rescue:+3.3V-RESCUE-Arduino_Mini-Arduino_Mini-rescue #PWR06
 U 1 1 5B0C2071
 P 9400 750
@@
 $EndComp
 Text Notes 875  -175 0    168  ~ 34
-Change TPS63031 footprint\nShorten last antenna segment\nDuplicate the antenna layout on second layer\nChange ground symbols\n
+ToDo:\nChange ground symbols\n
 $EndSCHEMATC
